File: contact-block-v4.kicad_sch (KiCad schematic)
At the start: 10 parts, among them J1 629105136821, J2 M06SIP, J3 MPT2, U1 PIC16F1459-I_SS

Commit message: Save schematic changes
Connections:
- net GND: now also J1.S1 (SHIELD), J1.S2 (SHIELD), J1.S3 (SHIELD), J1.S4 (SHIELD); no longer J1.SHELL (SHIELD), J1.SHELL1 (SHIELD), J1.SHELL2 (SHIELD), J1.SHELL3 (SHIELD)
- net at U1.8 (RC6): now also D1.2 (C); no longer D1.C
- net at R1.1: now also D1.1 (A); no longer D1.A

Commit message: Add parts and gerbers
Parts:
- C1: manf# (none) -> CAP CER 0.47UF 50V X7R 1206
- C2: manf# (none) -> C1206C104K5RAC7800
- C3: manf# (none) -> C1210F105K4RACTU
- D1: manf# (none) -> AA3528SURSK
- D2: manf# (none) -> TPD2E2U06QDBZRQ1
- J1: manf# (none) -> 629105136821
- J2, J3: DNP (none) -> ...
- R1: manf# (none) -> RT1206FRE071KL
- U1: manf# (none) -> PIC16F1459T-I/SS
Changed lines of the file:
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@@
+      (effects (font (size 1.27 1.27)) hide)
+    )
+    (property "DNP" "..." (id 4) (at 175.26 50.8 0)
       (effects (font (size 1.27 1.27)) hide)
     )
@@
       (effects (font (size 1.27 1.27)) hide)
     )
+    (property "DNP" "..." (id 4) (at 175.26 55.88 0)
+      (effects (font (size 1.27 1.27)) hide)
+    )
   )
   (symbol (lib_id "contact-block-v4-eagle-import:R-US_R1206") (at 81.28 45.72 0) (mirror y) (unit 1)
@@
       (effects (font (size 1.778 1.5113)) (justify left bottom) hide)
     )
+    (property "manf#" "	RT1206FRE071KL" (id 4) (at 81.28 45.72 0)
+      (effects (font (size 1.27 1.27)) hide)
+    )
   )
   (symbol (lib_id "contact-block-v4-eagle-import:LEDKA-3528ASYC") (at 91.44 45.72 90) (mirror x) (unit 1)
@@
       (effects (font (size 1.27 1.27)) hide)
     )
+    (property "manf#" "AA3528SURSK" (id 4) (at 91.44 45.72 0)
+      (effects (font (size 1.27 1.27)) hide)
+    )
   )
   (symbol (lib_id "contact-block-v4-eagle-import:C-USC1210") (at 101.6 99.06 0) (unit 1)
@@
       (effects (font (size 1.778 1.5113)) (justify left bottom) hide)
     )
+    (property "manf#" "C1210F105K4RACTU" (id 4) (at 101.6 99.06 0)
+      (effects (font (size 1.27 1.27)) hide)
+    )
   )
   (symbol (lib_id "contact-block-v4-eagle-import:C-USC1206K") (at 119.38 99.06 0) (unit 1)
@@
       (effects (font (size 1.778 1.5113)) (justify left bottom) hide)
     )
+    (property "manf#" "C1206C104K5RAC7800" (id 4) (at 119.38 99.06 0)
+      (effects (font (size 1.27 1.27)) hide)
+    )
   )
   (symbol (lib_id "contact-block-v4-eagle-import:C-USC1206K") (at 190.5 40.64 0) (unit 1)
@@
       (effects (font (size 1.778 1.5113)) (justify left bottom) hide)
     )
+    (property "manf#" "CAP CER 0.47UF 50V X7R 1206" (id 4) (at 190.5 40.64 0)
+      (effects (font (size 1.27 1.27)) hide)
+    )
   )
   (symbol (lib_id "contact-block-v4-eagle-import:M06SIP") (at 154.94 96.52 0) (mirror x) (unit 1)
@@
       (effects (font (size 1.27 1.27)) hide)
     )
+    (property "DNP" "..." (id 4) (at 154.94 96.52 0)
+      (effects (font (size 1.27 1.27)) hide)
+    )
   )
   (symbol (lib_id "contact-block-v4-eagle-import:629105136821") (at 238.76 33.02 0) (mirror x) (unit 1)
@@
       (effects (font (size 1.27 1.27)) hide)
     )
+    (property "manf#" "629105136821" (id 4) (at 238.76 33.02 0)
+      (effects (font (size 1.27 1.27)) hide)
+    )
   )
   (symbol (lib_id "contact-block-v4-eagle-import:TPD2E2U06QDBZRQ1") (at 200.66 78.74 0) (unit 1)
@@
       (effects (font (size 1.27 1.27)) hide)
     )
+    (property "manf#" "TPD2E2U06QDBZRQ1" (id 4) (at 200.66 78.74 0)
+      (effects (font (size 1.27 1.27)) hide)
+    )
   )
   (symbol (lib_id "contact-block-v4-eagle-import:PIC16F1459-I_SS") (at 104.14 55.88 0) (unit 1)
@@
       (effects (font (size 1.27 1.27)) hide)
     )
+    (property "manf#" "PIC16F1459T-I/SS" (id 4) (at 104.14 55.88 0)
+      (effects (font (size 1.27 1.27)) hide)
+    )
